Commit message: feat: reorganize workspace structure and add README with images

File: src/mower_bot_description/urdf/mower_core.xacro (robot description, xacro)
@@ -5,5 +5,5 @@
     <xacro:property name="base_y" value="0.60"/>
     <xacro:property name="base_z" value="0.14"/>
-    <xacro:property name="track_offset_y" value="0.33"/>
+    <xacro:property name="track_offset_y" value="0.25"/>
     <xacro:property name="drive_wheel_radius" value="0.05"/>
     <xacro:property name="drive_wheel_width" value="0.05"/>
